File: electronics/ChristmasCard/ChristmasCard.kicad_pcb (KiCad board)
At the start: 2 copper layers, 99.1 x 99.1 mm, 44 parts, among them J1 AVR-ISP-6, SW1 SW_Push, U1 LM78L05_TO92, U2 TAR5Sxx, U3 ATtiny24A-SSU

Commit message: Added kicad files.
Parts:
- removed D11, D12, D13, D14, D15, D16, D17, D18, D19: LED, LED_THT:LED_D5.0mm
- removed the R2 at (55.2, 59.7)
- removed the R3 at (95.9, 130.2)
- removed SW1: SW_Push, Button_Switch_THT:SW_CW_GPTS203211B
- moved C4 84.1 mm to (44.5, 104.8), turned to 90 degrees
- moved U2 82.5 mm to (50.8, 104.1)
- moved C2 75.5 mm to (57.1, 104.8), turned to 90 degrees
- moved R3 68.9 mm to (18.4, 104.1)
- moved C3 61.7 mm to (38.7, 85.1)
- moved C1 39.2 mm to (47.0, 60.3)
- moved C5 35.9 mm to (57.8, 85.1)
- moved R4 30.7 mm to (73.0, 104.8)
- moved R5 26.1 mm to (59.7, 65.4)
- moved D1 23.3 mm to (34.9, 89.5), turned to 180 degrees
- moved D21 23.1 mm to (6.99, 103.5)
- moved D27 23.1 mm to (89.5, 103.5)
- moved D25 18.2 mm to (62.9, 103.5)
- moved D23 18.0 mm to (35.6, 103.5)
- moved D26 14.6 mm to (76.8, 97.2)
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- renumbered R4 to R2, R5 to R3, R6 to R4, R7 to R5
Connections:
- D21 pad 2: Net-(D11-Pad2) -> Net-(D21-Pad2)
- D22 pad 1: Net-(D22-Pad1) -> Net-(D21-Pad1)
- D22 pad 2: Net-(D11-Pad2) -> Net-(D22-Pad2)
- D23 pad 1: Net-(D22-Pad1) -> Net-(D21-Pad1)
- D23 pad 2: Net-(D12-Pad2) -> Net-(D23-Pad2)
- D24 pad 1: Net-(D22-Pad1) -> Net-(D21-Pad1)
- D24 pad 2: Net-(D13-Pad2) -> Net-(D24-Pad2)
- D25 pad 1: Net-(D22-Pad1) -> Net-(D25-Pad1)
- D25 pad 2: Net-(D14-Pad2) -> Net-(D25-Pad2)
- D26 pad 1: Net-(D22-Pad1) -> Net-(D25-Pad1)
- D26 pad 2: Net-(D15-Pad2) -> Net-(D26-Pad2)
- D27 pad 1: Net-(D16-Pad1) -> Net-(D25-Pad1)
- D27 pad 2: Net-(D11-Pad2) -> Net-(D24-Pad2)
- D31 pad 1: Net-(D31-Pad1) -> Net-(D25-Pad1)
- D31 pad 2: Net-(D11-Pad2) -> Net-(D21-Pad2)
- D32 pad 1: Net-(D31-Pad1) -> Net-(D32-Pad1)
- D32 pad 2: Net-(D12-Pad2) -> Net-(D21-Pad2)
- D33 pad 1: Net-(D31-Pad1) -> Net-(D32-Pad1)
- D33 pad 2: Net-(D13-Pad2) -> Net-(D25-Pad2)
- D34 pad 1: Net-(D31-Pad1) -> Net-(D32-Pad1)
- D34 pad 2: Net-(D14-Pad2) -> Net-(D26-Pad2)
- D35 pad 1: Net-(D31-Pad1) -> Net-(D32-Pad1)
- D35 pad 2: Net-(D15-Pad2) -> Net-(D24-Pad2)
- D41 pad 1: Net-(D21-Pad1) -> Net-(D41-Pad1)
- D41 pad 2: Net-(D12-Pad2) -> Net-(D21-Pad2)
- D42 pad 1: Net-(D21-Pad1) -> Net-(D41-Pad1)
- D42 pad 2: Net-(D13-Pad2) -> Net-(D25-Pad2)
- D43 pad 1: Net-(D21-Pad1) -> Net-(D41-Pad1)
- D43 pad 2: Net-(D14-Pad2) -> Net-(D26-Pad2)
- D51 pad 1: Net-(D21-Pad1) -> Net-(D41-Pad1)
- D51 pad 2: Net-(D15-Pad2) -> Net-(D24-Pad2)
- J1 pad 1: Net-(D21-Pad1) -> Net-(D32-Pad1)
- J1 pad 3: Net-(J1-Pad3) -> Net-(D41-Pad1)
- J1 pad 4: Net-(D31-Pad1) -> Net-(D25-Pad1)
- R2 pad 2: Net-(D12-Pad2) -> Net-(D21-Pad2)
- R3 pad 2: Net-(D13-Pad2) -> Net-(D25-Pad2)
- R4 pad 2: Net-(D14-Pad2) -> Net-(D26-Pad2)
- R5 pad 2: Net-(D15-Pad2) -> Net-(D24-Pad2)
- U3 pad 2: Net-(D16-Pad1) -> Net-(U3-Pad2)
- U3 pad 6: Net-(D22-Pad1) -> Net-(D21-Pad1)
- U3 pad 7: Net-(D31-Pad1) -> Net-(D25-Pad1)
- U3 pad 8: Net-(D21-Pad1) -> Net-(D32-Pad1)
- U3 pad 9: Net-(J1-Pad3) -> Net-(D41-Pad1)
Routing:
- net Net-(CONN1-Pad1): track 0.00 -> 4.49 mm
- added copper zone on B.Cu, net GND
Other:
- outline, holes or cut-outs redrawn
