File: electronics/ChristmasCard/ChristmasCard.sch (KiCad schematic (older format))
At the start: 44 parts, among them J1 AVR-ISP-6, SW1 SW_Push, U1 LM78L05_TO92, U2 TAR5Sxx, U3 ATtiny24A-SSU

Commit message: Added kicad files.
Parts:
- removed D11, D12, D13, D14, D15, D16, D17, D18, D19: LED, LED_THT:LED_D5.0mm, symbol Device:LED_Small
- removed R2: 100K, Resistor_THT:R_Axial_DIN0207_L6.3mm_D2.5mm_P10.16mm_Horizontal, symbol Device:R_Small_US
- removed R3: 3K, Resistor_THT:R_Axial_DIN0207_L6.3mm_D2.5mm_P10.16mm_Horizontal, symbol Device:R_Small_US
- removed SW1: SW_Push, Button_Switch_THT:SW_CW_GPTS203211B, symbol Switch:SW_Push
- renumbered R4 to R2, R5 to R3, R6 to R4, R7 to R5
Connections:
- wire segments 157 -> 118
Other:
- moved on the sheet: D21, D22, D23, D24, D25, D26, D27, D31
